Commit message: Purposely enlarge the vacuum gripper to ensure being displayed in Gazebo #1.
Signed-off-by: Eric Dong <eric.dongxx@gmail.com>

File: robot_description/vacuum_gripper.urdf.xacro (robot description, xacro)
@@ -7,5 +7,5 @@
       <origin rpy="0 0 0" xyz="0 0 0"/>
       <geometry>
-        <cylinder radius="0.005" length="0.01"/>
+        <cylinder radius="0.05" length="0.02"/>
       </geometry>
       <material name="transparent">
@@ -21,5 +21,5 @@
   <joint name="gripper_joint" type="revolute">
     <axis xyz="1 0 0" />
-    <parent link="${prefix}ee_link" />
+    <parent link="${prefix}wrist_3_link" />
     <child link="${prefix}vacuum_gripper" />
     <origin rpy="0 1.5708 0" xyz="0.01 0.0125 0" />
