Commit message: Add robotiq_85_gripper into rendering in Gazebo. But corresponding ROS controller not implemented, dangling gripper now.. (Cannot compile with Gazebo 9)
Signed-off-by: Eric Dong <eric.dongxx@gmail.com>

File: robot_description/ur10_robot_test.urdf.xacro (robot description, xacro)
@@ -13,4 +13,9 @@
   <!-- kinect sensor -->
   <xacro:include filename="$(find ur_test)/robot_description/kinect.urdf.xacro" />
+  <!-- Robotiq gripper -->
+  <xacro:include filename="$(find robotiq_85_description)/urdf/robotiq_85_gripper.urdf.xacro"/>
+  <xacro:robotiq_85_gripper prefix="" parent="gripper_extender_link">
+    <origin xyz="0.1 0 0" rpy="${M_PI/2} -${M_PI/2} 0" />
+  </xacro:robotiq_85_gripper>
   <!-- arm -->
   <xacro:ur10_robot prefix="" joint_limited="false"/>

Commit message: Change location and rotation of the gripper to fit more into the extender link.
Signed-off-by: Eric Dong <eric.dongxx@gmail.com>

File: robot_description/ur10_robot_test.urdf.xacro (robot description, xacro)
@@ -16,5 +16,5 @@
   <xacro:include filename="$(find robotiq_85_description)/urdf/robotiq_85_gripper.urdf.xacro"/>
   <xacro:robotiq_85_gripper prefix="" parent="gripper_extender_link">
-    <origin xyz="0.1 0 0" rpy="${M_PI/2} -${M_PI/2} 0" />
+    <origin xyz="0.218 0 0" rpy="${M_PI/2} -${M_PI/2} ${M_PI/2}" />
   </xacro:robotiq_85_gripper>
   <!-- arm -->
